File: BEAMal_Rev1.kicad_pcb (KiCad board)
At the start: 2 copper layers, 438 x 160.5 mm, 131 parts, among them J1 CONN_CAP_IBM_F, J2 CONN_CAP_IBM_F

Commit message: Push after changes #1
Routing:
- net COL_1: track 285.0 -> 320.7 mm
- net COL_2: track 306.4 -> 316.2 mm
- net COL_9: track 327.9 -> 321.7 mm
- net ROW_6: track 783.3 -> 781.4 mm
- net ROW_5: track 800.8 -> 801.8 mm
