File: BEAMal_Rev1.kicad_pcb (KiCad board)
At the start: 2 copper layers, 438 x 160.5 mm, 131 parts, among them J1 CONN_CAP_IBM_F, J2 CONN_CAP_IBM_F

Commit message: Fixes #2
UPDATED gerbers
Parts:
- turned SW_02 to 180 degrees
Routing:
- net ROW_8: track 701.1 -> 730.6 mm
- net ROW_1: track 821.1 -> 843.4 mm
- net COL_9: track 321.7 -> 336.7 mm
- net COL_1: track 320.7 -> 312.7 mm
- net ROW_7: track 759.6 -> 755.8 mm
- net ROW_6: track 781.4 -> 778.6 mm
- net COL_5: track 198.3 -> 199.8 mm
- net ROW_5: track 801.8 -> 800.7 mm

Commit message: push update #3
Parts:
- moved COL_7_TP15 7.61 mm to (324.2, 259.9)
Routing:
- net COL_9: track 336.7 -> 374.4 mm
- net COL_4: track 230.3 -> 256.6 mm
- net COL_8: track 264.1 -> 281.1 mm
- net COL_3: track 272.8 -> 285.2 mm
- net COL_C: track 368.0 -> 378.7 mm
- net COL_6: track 213.4 -> 223.1 mm
- net COL_5: track 199.8 -> 190.1 mm
- net COL_7: track 261.7 -> 263.0 mm
