File: BEAMal_Rev1.kicad_pcb (KiCad board)
At the start: 2 copper layers, 438 x 160.5 mm, 131 parts, among them J1 CONN_CAP_IBM_F, J2 CONN_CAP_IBM_F

Commit message: Push Added Controller
Parts:
- added C1: 0U1, Capacitor_SMD:C_0805_2012Metric_Pad1.15x1.40mm_HandSolder, B.Cu at (188.3, 30.3)
- added C2: 0U1, Capacitor_SMD:C_0805_2012Metric_Pad1.15x1.40mm_HandSolder, B.Cu at (278.5, 31.6)
- added C3: 0U1, Capacitor_SMD:C_0805_2012Metric_Pad1.15x1.40mm_HandSolder, B.Cu at (201.3, 27.7)
- added C4: 0U1, Capacitor_SMD:C_0805_2012Metric_Pad1.15x1.40mm_HandSolder, B.Cu at (246.7, 31.5)
- added C6: 0U1, Capacitor_SMD:C_0805_2012Metric_Pad1.15x1.40mm_HandSolder, B.Cu at (209.3, 26.8)
- added C7: 0U1, Capacitor_SMD:C_0805_2012Metric_Pad1.15x1.40mm_HandSolder, B.Cu at (225.2, 26.6)
- added J3: EXPANSION HEADER, TH-XWhatsIt:PinHeader_2x03_P2.54mm_Vertical_3dhorizontal, F.Cu at (331.1, 34.8)
- added J6: MODEL F AT LOCKLIGHTS HEADER, TH-XWhatsIt:FAT_LockLightsConnector, F.Cu at (331.1, 45.2)
- added NT1: Net-Tie_4_Cross, NetTie:NetTie-4_THT_Pad1.0mm, F.Cu at (324.2, 23.1)
- added R1: 4K7, Resistor_SMD:R_0805_2012Metric_Pad1.15x1.40mm_HandSolder, B.Cu at (214.8, 26.6)
- added R10: 100k 1%, Resistor_SMD:R_0805_2012Metric_Pad1.15x1.40mm_HandSolder, B.Cu at (216.1, 36.1)
- added R11: 100k 1%, Resistor_SMD:R_0805_2012Metric_Pad1.15x1.40mm_HandSolder, B.Cu at (202.4, 32.6)
- added R12: 100k 1%, Resistor_SMD:R_0805_2012Metric_Pad1.15x1.40mm_HandSolder, B.Cu at (202.4, 36.1)
- added R13: 100k 1%, Resistor_SMD:R_0805_2012Metric_Pad1.15x1.40mm_HandSolder, B.Cu at (232.2, 32.7)
- added R14: 100k 1%, Resistor_SMD:R_0805_2012Metric_Pad1.15x1.40mm_HandSolder, B.Cu at (232.2, 36.1)
- added R15: 100k 1%, Resistor_SMD:R_0805_2012Metric_Pad1.15x1.40mm_HandSolder, B.Cu at (218.3, 29.2)
- added R16: 100k 1%, Resistor_SMD:R_0805_2012Metric_Pad1.15x1.40mm_HandSolder, B.Cu at (218.3, 33.8)
- added R17: 330, Resistor_SMD:R_0805_2012Metric_Pad1.15x1.40mm_HandSolder, B.Cu at (332.8, 42.9)
- added R18: 330, Resistor_SMD:R_0805_2012Metric_Pad1.15x1.40mm_HandSolder, B.Cu at (326.2, 53.1)
- added R19: 330, Resistor_SMD:R_0805_2012Metric_Pad1.15x1.40mm_HandSolder, B.Cu at (326.2, 51.0)
- added R2: 1K, Resistor_SMD:R_0805_2012Metric_Pad1.15x1.40mm_HandSolder, B.Cu at (220.1, 26.6)
- added R3: 20K, Resistor_SMD:R_0805_2012Metric_Pad1.15x1.40mm_HandSolder, B.Cu at (197.0, 33.0)
- added R4: 20K, Resistor_SMD:R_0805_2012Metric_Pad1.15x1.40mm_HandSolder, B.Cu at (191.7, 33.0)
- added R5: 4K7, Resistor_SMD:R_0805_2012Metric_Pad1.15x1.40mm_HandSolder, B.Cu at (197.0, 35.6)
- added R6: Not Mounted, Resistor_SMD:R_0805_2012Metric_Pad1.15x1.40mm_HandSolder, B.Cu at (303.0, 33.8)
- added R7: Not Mounted, Resistor_SMD:R_0805_2012Metric_Pad1.15x1.40mm_HandSolder, B.Cu at (306.7, 33.8)
- added R8: Not Mounted, Resistor_SMD:R_0805_2012Metric_Pad1.15x1.40mm_HandSolder, B.Cu at (310.6, 33.8)
- added R9: 100k 1%, Resistor_SMD:R_0805_2012Metric_Pad1.15x1.40mm_HandSolder, B.Cu at (216.1, 31.5)
- added TP1: Dac Output, TestPoint:TestPoint_Pad_D1.0mm, B.Cu at (184.1, 30.1)
- added TP2: Threshold Voltage, TestPoint:TestPoint_Pad_D1.0mm, B.Cu at (184.2, 27.5)
- added U1: MCP4921-E, Package_SO:SOIC-8_3.9x4.9mm_P1.27mm, B.Cu at (195.2, 28.6)
- added U2: LM339A, Package_SO:SOIC-14_3.9x8.7mm_P1.27mm, B.Cu at (209.3, 32.6)
- added U3: 74AHC595, Package_SO:SOIC-16_3.9x9.9mm_P1.27mm, B.Cu at (285.9, 31.5)
- added U4: 74AHC595, Package_SO:SOIC-16_3.9x9.9mm_P1.27mm, B.Cu at (254.2, 31.5)
- added U5: ProMicro, promicro:ProMicro, F.Cu at (319.3, 22.2)
- added U6: LM339A, Package_SO:SOIC-14_3.9x8.7mm_P1.27mm, B.Cu at (225.2, 32.6)
- J1: value CONN_CAP_IBM_F -> Model F Ribbon Cable; footprint lib_fp:CONN_CAP_IBM_F -> TH-XWhatsIt:Model_F_3.96mm_pitch_footprint
- J2: value CONN_CAP_IBM_F -> PadsToShort; footprint beamspring card edge:BEAMSPRING-CARD-EDGE -> TH-XWhatsIt:PadsToShort; moved to B.Cu
- moved J2 121.5 mm to (329.4, 26.5)
- moved J1 86.0 mm to (195.5, 39.2)
- moved G*** 58.7 mm to (377.7, 91.5)
Connections:
- J1 pad 1: GND -> (no net)
- J1 pad 10: ROW_8 -> (no net)
- J1 pad 11: GND -> (no net)
- J1 pad 12: GND -> (no net)
- J1 pad 13: COL_1 -> (no net)
- J1 pad 14: COL_2 -> (no net)
- J1 pad 15: COL_3 -> (no net)
- J1 pad 16: COL_4 -> (no net)
- J1 pad 17: COL_5 -> (no net)
- J1 pad 18: COL_6 -> (no net)
- J1 pad 19: COL_7 -> (no net)
- J1 pad 2: GND -> (no net)
- J1 pad 20: COL_8 -> (no net)
- J1 pad 21: COL_9 -> (no net)
- J1 pad 22: COL_A -> (no net)
- J1 pad 23: COL_B -> (no net)
- J1 pad 24: COL_C -> (no net)
- J1 pad 25: COL_D -> (no net)
- J1 pad 26: COL_E -> (no net)
- J1 pad 27: COL_F -> (no net)
- J1 pad 28: COL_G -> (no net)
- J1 pad 29: GND -> (no net)
- J1 pad 3: ROW_1 -> (no net)
- J1 pad 30: GND -> (no net)
- J1 pad 4: ROW_2 -> (no net)
- J1 pad 5: ROW_3 -> (no net)
- J1 pad 6: ROW_4 -> (no net)
- J1 pad 7: ROW_5 -> (no net)
- J1 pad 8: ROW_6 -> (no net)
- J1 pad 9: ROW_7 -> (no net)
- J2 pad 1: GND -> (no net)
- J2 pad 2: GND -> (no net)
Routing:
- net (no net): track 0.00 -> 2951.3 mm, vias 0 -> 395
- net COL_C: track 368.0 -> 142.4 mm
- net COL_B: track 353.8 -> 141.9 mm
- net COL_A: track 338.3 -> 140.7 mm
- net ROW_7: track 759.6 -> 592.2 mm
- net ROW_6: track 783.3 -> 617.5 mm
- net ROW_5: track 800.8 -> 639.4 mm
- net ROW_8: track 701.1 -> 546.1 mm
- net COL_9: track 327.9 -> 177.0 mm
- net ROW_4: track 784.4 -> 634.0 mm
- net ROW_3: track 798.0 -> 651.5 mm
- net ROW_2: track 810.6 -> 668.1 mm
- net ROW_1: track 821.1 -> 682.6 mm
- net COL_8: track 264.1 -> 152.7 mm
- net COL_7: track 261.7 -> 183.7 mm
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- added copper zone on B.Cu, net (none)
- added copper zone on F.Cu, net (none)
- removed copper zone on B.Cu, net GND
- removed copper zone on F.Cu, net GND
Other:
- board text added: "JLCJLCJLCJLC"
- board text added: "↑↑↑ Pins for: F AT/122/Unsaver keyboards ↑↑↑"

Commit message: puah
Parts:
- added J1: CONN_CAP_IBM_F, lib_fp:CONN_CAP_IBM_F, F.Cu at (191.4, 144.7)
- added J2: CONN_CAP_IBM_F, beamspring card edge:BEAMSPRING-CARD-EDGE, F.Cu at (248.8, 138.3)
- moved G*** 76.6 mm to (344.8, 160.7)
- moved COL_7_TP15 20.3 mm to (322.7, 279.5)
- moved COL_1_TP9 19.7 mm to (93.2, 279.5)
- moved COL_2_TP10 19.7 mm to (111.7, 280.0)
- moved COL_4_TP12 19.7 mm to (196.7, 279.5)
- moved COL_5_TP13 19.7 mm to (259.6, 280.0)
- moved COL_8_TP16 19.7 mm to (340.8, 280.0)
- moved COL_9_TP17 19.7 mm to (370.8, 279.8)
- moved H11 19.7 mm to (92.9, 289.3)
- moved H2 19.7 mm to (250.5, 289.3)
- moved H4 19.7 mm to (407.3, 289.3)
- moved H7 19.7 mm to (83.3, 289.3)
- moved H9 19.7 mm to (483.5, 289.3)
- moved COL_B_TP19 19.7 mm to (474.9, 279.8)
- moved H6 19.7 mm to (416.9, 289.3)
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Routing:
- net COL_C: track 142.4 -> 378.7 mm
- net COL_B: track 141.9 -> 353.8 mm
- net COL_A: track 140.7 -> 338.3 mm
- net COL_9: track 177.0 -> 374.4 mm
- net ROW_8: track 546.1 -> 730.6 mm
- net ROW_7: track 592.2 -> 755.8 mm
- net ROW_5: track 639.4 -> 800.7 mm
- net ROW_6: track 617.5 -> 778.6 mm
- net ROW_1: track 682.6 -> 843.4 mm
- net ROW_4: track 634.0 -> 784.4 mm
- net ROW_3: track 651.5 -> 798.0 mm
- net ROW_2: track 668.1 -> 810.6 mm
- net COL_8: track 152.7 -> 281.1 mm
- net COL_7: track 183.7 -> 263.0 mm
- net COL_4: track 181.6 -> 256.6 mm
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Other:
- board text added: "G***"
- board text added: "LOGO"

Commit message: update
Parts:
- removed the J1 at (191.4, 144.7)
- removed the J2 at (248.8, 138.3)
- moved COL_6_TP14 28.2 mm to (260.8, 288.2)
- moved COL_7_TP15 28.2 mm to (295.8, 287.8)
- moved ROW_1_TP1 28.2 mm to (481.3, 268.9)
- moved ROW_4_TP4 28.2 mm to (482.0, 218.2)
- moved SW_21 28.2 mm to (260.4, 200.1)
- moved SW_22 28.2 mm to (279.5, 200.1)
- moved SW_51 28.2 mm to (293.9, 238.2)
- moved SW_52 28.2 mm to (313.0, 238.2)
- moved SW_61 28.2 mm to (265.4, 257.3)
- moved SW_62 28.2 mm to (284.5, 257.3)
- moved SW_69 28.2 mm to (308.5, 276.3)
- moved SW_74 28.2 mm to (451.9, 181.1)
- moved SW_75 28.2 mm to (471.0, 181.1)
- moved SW_78 28.2 mm to (451.9, 200.1)
- moved SW_79 28.2 mm to (471.0, 200.1)
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
Commit message: giving up on this
Parts:
- removed J1: Model F Ribbon Cable, TH-XWhatsIt:Model_F_3.96mm_pitch_footprint
- removed R6: Not Mounted, Resistor_SMD:R_0805_2012Metric_Pad1.15x1.40mm_HandSolder
- C1, C2, C3, C4, C6, C7: footprint Capacitor_SMD:C_0805_2012Metric_Pad1.15x1.40mm_HandSolder -> capacitor_smd:C_0805_2012Metric_Pad1.15x1.40mm_HandSolder
- moved J2 129.2 mm to (276.6, 144.3)
- moved J6 129.2 mm to (278.3, 163.1)
- moved R17 129.2 mm to (280.0, 160.8)
- moved J3 129.2 mm to (278.3, 152.7)
- moved NT1 129.2 mm to (271.4, 140.9)
- moved R18 129.2 mm to (273.4, 171.0)
- moved R19 129.2 mm to (273.4, 168.9)
- moved R7 129.2 mm to (253.9, 151.7)
- moved R8 129.2 mm to (257.8, 151.7)
- moved U5 129.2 mm to (266.4, 140.1)
- moved C2 117.4 mm to (234.9, 140.6)
- moved U3 117.4 mm to (242.3, 140.5)
- moved C3 114.4 mm to (182.8, 140.6)
- moved R13 114.4 mm to (213.7, 145.6)
- moved R15 114.4 mm to (199.8, 142.1)
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Connections:
- C1 pad 1: (no net) -> GND
- C1 pad 2: (no net) -> +5VD
- C2 pad 1: (no net) -> GND
- C2 pad 2: (no net) -> +5VD
- C3 pad 1: (no net) -> GND
- C3 pad 2: (no net) -> +5VA
- C4 pad 1: (no net) -> GND
- C4 pad 2: (no net) -> +5VD
- C6 pad 1: (no net) -> GND
- C6 pad 2: (no net) -> +5VA
- C7 pad 1: (no net) -> GND
- C7 pad 2: (no net) -> +5VA
- J2 pad 1: (no net) -> RST
- J2 pad 2: (no net) -> GND
- J3 pad 1: (no net) -> +5VL
- J3 pad 2: (no net) -> HEADER3_ENABLE
- J3 pad 3: (no net) -> HEADER1_NUMLCK
- J3 pad 4: (no net) -> HEADER4_TRIGGER
- J3 pad 5: (no net) -> HEADER2_CAPSLCK
- J3 pad 6: (no net) -> GND
- J6 pad 2: (no net) -> Net-(J6-Pin_2)
- J6 pad 3: (no net) -> unconnected-(J6-Pin_3)
- J6 pad 4: (no net) -> Net-(J6-Pin_4)
- J6 pad 5: (no net) -> GND
- J6 pad 6: (no net) -> Net-(J6-Pin_6)
- J6 pad 7: (no net) -> +5VL
- J6 pad 8: (no net) -> unconnected-(J6-Pin_8)
- NT1 pad 1: (no net) -> VCC
- NT1 pad 2: (no net) -> +5VL
- NT1 pad 3: (no net) -> +5VA
- NT1 pad 4: (no net) -> +5VD
- R1 pad 1: (no net) -> +5VA
- R1 pad 2: (no net) -> BIAS
- R10 pad 1: (no net) -> BIAS
- R10 pad 2: (no net) -> SENSE3
- R11 pad 1: (no net) -> BIAS
- R11 pad 2: (no net) -> SENSE1
- R12 pad 1: (no net) -> BIAS
- R12 pad 2: (no net) -> SENSE2
- R13 pad 1: (no net) -> BIAS
- R13 pad 2: (no net) -> SENSE8
- R14 pad 1: (no net) -> BIAS
- R14 pad 2: (no net) -> SENSE6
- R15 pad 1: (no net) -> BIAS
- R15 pad 2: (no net) -> SENSE5
- R16 pad 1: (no net) -> BIAS
- R16 pad 2: (no net) -> SENSE7
- R17 pad 1: (no net) -> Net-(J6-Pin_2)
- R17 pad 2: (no net) -> HEADER2_CAPSLCK
- R18 pad 1: (no net) -> Net-(J6-Pin_4)
- R18 pad 2: (no net) -> HEADER1_NUMLCK
- R19 pad 1: (no net) -> Net-(J6-Pin_6)
- R19 pad 2: (no net) -> HEADER5_SCRLCK
- R2 pad 1: (no net) -> GND
- R2 pad 2: (no net) -> BIAS
- R3 pad 1: (no net) -> SETPOINT
- R3 pad 2: (no net) -> +5VA
- R4 pad 1: (no net) -> SETPOINT
- R4 pad 2: (no net) -> Net-(U1-VoutA)
- R5 pad 1: (no net) -> GND
- R5 pad 2: (no net) -> SETPOINT
- R7 pad 1: (no net) -> HEADER5_SCRLCK
- R7 pad 2: (no net) -> GND
- R8 pad 1: (no net) -> Net-(U5-PB3(D14,MISO))
- R8 pad 2: (no net) -> GND
- R9 pad 1: (no net) -> BIAS
- R9 pad 2: (no net) -> SENSE4
- TP1 pad 1: (no net) -> Net-(U1-VoutA)
- TP2 pad 1: (no net) -> SETPOINT
- U1 pad 1: (no net) -> +5VD
- U1 pad 2: (no net) -> ~{SELECTDAC}
- U1 pad 3: (no net) -> CLOCK
- U1 pad 4: (no net) -> MOSI
- U1 pad 5: (no net) -> GND
- U1 pad 6: (no net) -> +5VA
- U1 pad 7: (no net) -> GND
- U1 pad 8: (no net) -> Net-(U1-VoutA)
- U2 pad 1: (no net) -> ROW3
- U2 pad 10: (no net) -> SETPOINT
- U2 pad 11: (no net) -> SENSE1
- U2 pad 12: (no net) -> GND
- U2 pad 13: (no net) -> ROW1
- U2 pad 14: (no net) -> ROW2
- U2 pad 2: (no net) -> ROW4
- U2 pad 3: (no net) -> +5VA
- U2 pad 4: (no net) -> SETPOINT
- U2 pad 5: (no net) -> SENSE4
- U2 pad 6: (no net) -> SETPOINT
- U2 pad 7: (no net) -> SENSE3
- U2 pad 8: (no net) -> SETPOINT
- U2 pad 9: (no net) -> SENSE2
- U3 pad 1: (no net) -> COL2
- U3 pad 10: (no net) -> +5VD
- U3 pad 11: (no net) -> CLOCK
- U3 pad 12: (no net) -> LOADCOL
- U3 pad 13: (no net) -> GND
- U3 pad 14: (no net) -> MOSI
- U3 pad 15: (no net) -> COL1
- U3 pad 16: (no net) -> +5VD
- U3 pad 2: (no net) -> COL3
- U3 pad 3: (no net) -> COL4
- U3 pad 4: (no net) -> COL5
- U3 pad 5: (no net) -> COL6
- U3 pad 6: (no net) -> COL7
- U3 pad 7: (no net) -> COL8
- U3 pad 8: (no net) -> GND
- U3 pad 9: (no net) -> SERIALOUT1
- U4 pad 1: (no net) -> COL10
- U4 pad 10: (no net) -> +5VD
- U4 pad 11: (no net) -> CLOCK
- U4 pad 12: (no net) -> LOADCOL
- U4 pad 13: (no net) -> GND
- U4 pad 14: (no net) -> SERIALOUT1
- U4 pad 15: (no net) -> COL9
- U4 pad 16: (no net) -> +5VD
- U4 pad 2: (no net) -> COL11
- U4 pad 3: (no net) -> COL12
- U4 pad 4: (no net) -> COL13
- U4 pad 5: (no net) -> COL14
- U4 pad 6: (no net) -> COL15
- U4 pad 7: (no net) -> COL16
- U4 pad 8: (no net) -> GND
- U4 pad 9: (no net) -> unconnected-(U4-QH')
- U5 pad 1: (no net) -> HEADER3_ENABLE
- U5 pad 10: (no net) -> HEADER2_CAPSLCK
- U5 pad 11: (no net) -> ROW5
- U5 pad 12: (no net) -> ROW6
- U5 pad 13: (no net) -> HEADER5_SCRLCK
- U5 pad 14: (no net) -> MOSI
- U5 pad 15: (no net) -> Net-(U5-PB3(D14,MISO))
- U5 pad 16: (no net) -> CLOCK
- U5 pad 17: (no net) -> LOADCOL
- U5 pad 18: (no net) -> ~{SELECTDAC}
- U5 pad 19: (no net) -> ROW8
- U5 pad 2: (no net) -> HEADER4_TRIGGER
- U5 pad 20: (no net) -> ROW7
- U5 pad 21: (no net) -> VCC
- U5 pad 22: (no net) -> RST
- U5 pad 23: (no net) -> GND
- U5 pad 24: (no net) -> unconnected-(U5-RAW)
- U5 pad 3: (no net) -> GND
- U5 pad 4: (no net) -> GND
- U5 pad 5: (no net) -> ROW2
- U5 pad 6: (no net) -> ROW1
- U5 pad 7: (no net) -> ROW4
- U5 pad 8: (no net) -> ROW3
- U5 pad 9: (no net) -> HEADER1_NUMLCK
- U6 pad 1: (no net) -> ROW6
- U6 pad 10: (no net) -> SETPOINT
- U6 pad 11: (no net) -> SENSE5
- U6 pad 12: (no net) -> GND
- U6 pad 13: (no net) -> ROW5
- U6 pad 14: (no net) -> ROW7
- U6 pad 2: (no net) -> ROW8
- U6 pad 3: (no net) -> +5VA
- U6 pad 4: (no net) -> SETPOINT
- U6 pad 5: (no net) -> SENSE8
- U6 pad 6: (no net) -> SETPOINT
- U6 pad 7: (no net) -> SENSE6
- U6 pad 8: (no net) -> SETPOINT
- U6 pad 9: (no net) -> SENSE7
Routing:
- net (no net): track 3023.3 -> 0.00 mm, vias 395 -> 341
- net COL_C: track 378.7 -> 153.9 mm
- net COL_B: track 353.8 -> 141.9 mm
- net COL_A: track 338.3 -> 140.7 mm
- net COL_1: track 312.7 -> 147.4 mm
- net COL_9: track 374.4 -> 223.2 mm
- net ROW_4: track 784.4 -> 634.0 mm
- net ROW_3: track 798.0 -> 651.5 mm
- net ROW_2: track 810.6 -> 668.1 mm
- net ROW_8: track 730.6 -> 588.6 mm
- net ROW_7: track 755.8 -> 616.1 mm
- net ROW_1: track 843.4 -> 704.9 mm
- net +5VA: track 0.00 -> 137.4 mm, vias 0 -> 6
- net ROW_6: track 778.6 -> 642.2 mm
- net ROW_5: track 800.7 -> 668.6 mm
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Other:
- board size 438 x 160.5 mm -> 438 x 165.6 mm
- board text removed: "↑↑↑ Pins for: F AT/122/Unsaver keyboards ↑↑↑"
