File: BEAMal_Rev1.kicad_sch (KiCad schematic)
At the start: 129 parts

Commit message: Push Added Controller
Parts:
- removed U (x2): (no value), symbol lib_sch:CONN_CAP_IBM_F
- added U (x6): (no value), symbol Device:C_Small
- added U (x10): (no value), symbol Comparator:LM339
- added U (x5): (no value), symbol Device:R_Small_US
- added U (x3): (no value), symbol Mechanical:MountingHole
- added U (x3): (no value), symbol Mechanical:MountingHole_Pad
- added U: (no value), symbol model_f_at_locklights_sym:Conn_02x04_Odd_Even
- added U (x2): (no value), symbol Connector_Generic:Conn_01x30
- added U (x14): (no value), symbol Device:R
- added U (x2): (no value), symbol Connector:TestPoint
- added U (x2): (no value), symbol 74xx:74HCT595
- added U: (no value), symbol Connector_Generic:Conn_02x03_Odd_Even
- added U: (no value), symbol Analog_DAC:MCP4921-EP
- added U: (no value), symbol SMDModelF-rescue:Net-Tie_4_Cross-Device
- added U: (no value), symbol Connector_Generic:Conn_01x02
- added U: (no value), symbol promicro:ProMicro
Connections:
- net GND: now also U.1, U.1, U.1, U.1, U.1, U.1, U.1, U.1, U.1, U.1, U.1, U.1 (Pin_1), U.11 (Pin_11), U.12 (Pin_12), U.13 (~{OE}), U.13 (~{OE}), U.2, U.2, U.2 (Pin_2), U.2 (Pin_2), U.22 (Pin_22), U.23 (GND), U.23 (Pin_23), U.24 (Pin_24), U.25 (Pin_25), U.26 (Pin_26), U.27 (Pin_27), U.28 (Pin_28), U.29 (Pin_29), U.29 (Pin_29), U.3 (GND), U.30 (Pin_30), U.30 (Pin_30), U.4 (GND), U.5 (Pin_5), U.5 (~{LDAC}), U.6 (Pin_6), U.7 (AVSS), U.8 (GND), U.8 (GND), U.9 (Pin_9)
- new net: U.1, U.2 (Pin_2)
- new net: U.1, U.4 (Pin_4)
- new net: U.1, U.6 (Pin_6)
- new net: U.1, U.2, U.8 (VoutA)
- new net: U.1, U.15 (PB3(D14,MISO))
- new net +5VA: U.1, U.2, U.2, U.2, U.2, U.3, U.6 (VrefA)
- new net +5VD: U.1, U.1 (VDD), U.10 (~{SRCLR}), U.10 (~{SRCLR}), U.16 (VCC), U.16 (VCC), U.2, U.2, U.2, U.4
- new net +5VL: U.1 (Pin_1), U.2, U.7 (Pin_7)
- new net BIAS: U.1, U.1, U.1, U.1, U.1, U.1, U.1, U.1, U.2, U.2
- new net CLOCK: U.11 (SRCLK), U.11 (SRCLK), U.16 (PB1(D15,SCLK)), U.3 (SCK)
- new net COL1: U.15 (QA), U.28 (Pin_28)
- new net COL10: U.1 (QB), U.16 (Pin_16), U.19 (Pin_19)
- new net COL11: U.15 (Pin_15), U.18 (Pin_18), U.2 (QC)
- new net COL12: U.14 (Pin_14), U.17 (Pin_17), U.3 (QD)
- new net COL13: U.13 (Pin_13), U.16 (Pin_16), U.4 (QE)
- new net COL14: U.12 (Pin_12), U.15 (Pin_15), U.5 (QF)
- new net COL15: U.11 (Pin_11), U.14 (Pin_14), U.6 (QG)
- new net COL16: U.10 (Pin_10), U.13 (Pin_13), U.7 (QH)
- new net COL2: U.1 (QB), U.27 (Pin_27)
- new net COL3: U.2 (QC), U.26 (Pin_26)
- new net COL4: U.25 (Pin_25), U.3 (QD)
- new net COL5: U.21 (Pin_21), U.24 (Pin_24), U.4 (QE)
- new net COL6: U.20 (Pin_20), U.23 (Pin_23), U.5 (QF)
- new net COL7: U.19 (Pin_19), U.22 (Pin_22), U.6 (QG)
- new net COL8: U.18 (Pin_18), U.21 (Pin_21), U.7 (QH)
- new net COL9: U.15 (QA), U.17 (Pin_17), U.20 (Pin_20)
- new net HEADER1_NUMLCK: U.2, U.3 (Pin_3), U.9 (PD7(D6,A7))
- new net HEADER2_CAPSLCK: U.10 (PE6(D7)), U.2, U.5 (Pin_5)
- new net HEADER3_ENABLE: U.1 (PD3(D1,TX)), U.2 (Pin_2)
- new net HEADER4_TRIGGER: U.2 (PD2(D0,RX)), U.4 (Pin_4)
- new net HEADER5_SCRLCK: U.1, U.13 (PB6(D10)), U.2, U.2
- new net LOADCOL: U.12 (RCLK), U.12 (RCLK), U.17 (PF7(D18,A0))
- new net MOSI: U.14 (PB2(D16,MOSI)), U.14 (SER), U.4 (SDI)
- new net ROW1: U.2, U.6 (PD0(D3,SCL))
- new net ROW2: U.2, U.5 (PD1(D2,SDA))
- new net ROW3: U.2, U.8 (PC6(D5))
- new net ROW4: U.2, U.7 (PD4(D4,A6))
- new net ROW5: U.11 (PB4(D8,A8)), U.2
- new net ROW6: U.12 (PB5(D9,A9)), U.2
- new net ROW7: U.2, U.20 (PF4(D21,A3))
- new net ROW8: U.19 (PF5(D20,A2)), U.2
- new net RST: U.1 (Pin_1), U.22 (RST)
- new net SENSE1: U.1 (Pin_1), U.2, U.3 (Pin_3), U.5 (+)
- new net SENSE2: U.2, U.2 (Pin_2), U.4 (Pin_4), U.5 (+)
- new net SENSE3: U.2, U.3 (Pin_3), U.5 (+), U.5 (Pin_5)
- new net SENSE4: U.2, U.4 (Pin_4), U.5 (+), U.6 (Pin_6)
- new net SENSE5: U.2, U.5 (+), U.5 (Pin_5), U.7 (Pin_7)
- new net SENSE6: U.2, U.5 (+), U.7 (Pin_7), U.9 (Pin_9)
- new net SENSE7: U.2, U.5 (+), U.6 (Pin_6), U.8 (Pin_8)
- new net SENSE8: U.10 (Pin_10), U.2, U.5 (+), U.8 (Pin_8)
- new net SERIALOUT1: U.14 (SER), U.9 (QH')
- new net SETPOINT: U.1, U.1, U.1, U.2, U.4 (-), U.4 (-), U.4 (-), U.4 (-), U.4 (-), U.4 (-), U.4 (-), U.4 (-)
- new net VCC: U.1, U.21 (VCC)
- new net ~{SELECTDAC}: U.18 (PF6(D19,A1)), U.2 (~{CS})
- no-connect marks 0 -> 4
Other:
- note added: "Copyright Rainy Day Plans. This documentation describes Open Hardware and is licensed under the CERN OHL v. 1.2. You may redistribute and modify this documentation under the terms of the CERN OHL v.1.2. (http://ohwr.org/cernohl). This documentation is distributed WITHOUT ANY EXPRESS OR IMPLIED WARRANTY, INCLUDING OF MERCHANTABILITY, SATISFACTORY QUALITY AND FITNESS FOR A PARTICULAR PURPOSE. Pleas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"
- note added: "NOTE1: pin B3 grounded will mean in the future that it's a controller needs to be driven differently by software, compared to the original TH Xwhatsit design. NOTE2: pin B6 can be an ADC input, so we may use it in the future to determine board version. Version is specified by selecting a voltage with a voltage divider. Note3: if versioning is enabled by pulling pin B3 low, HEADER5_SCRLCK must not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"
- note added: "Note: the Model F AT lights are in this order: (left -> right) Caps Lock Num Lock Note2: These are active-high signals. Scroll Lock"

Commit message: puah
Parts:
- removed U (x3): (no value), symbol Mechanical:MountingHole
- removed U (x3): (no value), symbol Mechanical:MountingHole_Pad
- removed U (x2): (no value), symbol Connector_Generic:Conn_01x30
